File: slime_tracker.kicad_sch (KiCad schematic)
At the start: 20 parts, among them CN1 SM05B-SRSS-TB (LF)(SN), SW1 MK-12C02-G020, U1 ICM-45686, U2 QMC6309, Y1 1532H-24.000JWVDTL

Commit message: Converted from global to project libraries
Parts:
- CN1: footprint Personal:CONN-SMD_SM05B-SRSS-TB-LF-SN -> Bert-Slime-PCB:CONN-SMD_SM05B-SRSS-TB-LF-SN; symbol SM05B-SRSS-TB-con:SM05B-SRSS-TB(LF)(SN) -> Bert-Slime-PCB:SM05B-SRSS-TB(LF)(SN)
- D1, D2: footprint PMEG3010ESBYL:SOD993_L1.0-W0.6-LS1.0-RD -> Bert-Slime-PCB:SOD993_L1.0-W0.6-LS1.0-RD; symbol PMEG3010ESBYL:PMEG3010ESBYL -> Bert-Slime-PCB:PMEG3010ESBYL
- SW1: footprint Personal:SW-SMD_MK-12C02-G020 -> Bert-Slime-PCB:SW-SMD_MK-12C02-G020; symbol MK-12C02-G020:MK-12C02-G020 -> Bert-Slime-PCB:MK-12C02-G020
- U1: footprint ICM_45686:IC_ICM-45686 -> Bert-Slime-PCB:IC_ICM-45686; symbol ICM-45686:ICM-45686 -> Bert-Slime-PCB:ICM-45686
- U2: footprint QMC6309-lib:X1-WLB0808-4_L0.8-W0.8-P0.40-TL -> Bert-Slime-PCB:X1-WLB0808-4_L0.8-W0.8-P0.40-TL; symbol QMC6309:QMC6309 -> Bert-Slime-PCB:QMC6309
- U3: footprint Personal:D1-Mini -> Bert-Slime-PCB:D1-Mini; symbol Personal_Library:D1_Mini -> Bert-Slime-PCB:D1_Mini; now in the parts list
- U4: footprint Personal:TP4056-USBC-MODULE -> Bert-Slime-PCB:TP4056-USBC-MODULE; symbol kicad-library:TP4056-USBC-Module -> Bert-Slime-PCB:TP4056-USBC-Module; now in the parts list
- Y1: footprint Personal:Crystal_SMD_3225-4Pin_3.2x2.5mm -> Crystal:Crystal_SMD_3225-4Pin_3.2x2.5mm; symbol Personal_Library:1532H-24.000JWVDTL -> Bert-Slime-PCB:1532H-24.000JWVDTL
Changed lines of the file:
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@@
 	)
 	(symbol
-		(lib_id "QMC6309:QMC6309")
+		(lib_id "Bert-Slime-PCB:QMC6309")
 		(at 237.49 137.16 0)
 		(unit 1)
@@
 			)
 		)
-		(property "Footprint" "QMC6309-lib:X1-WLB0808-4_L0.8-W0.8-P0.40-TL"
+		(property "Footprint" "Bert-Slime-PCB:X1-WLB0808-4_L0.8-W0.8-P0.40-TL"
 			(at 237.49 146.05 0)
 			(effects
@@
 	)
 	(symbol
-		(lib_id "ICM-45686:ICM-45686")
+		(lib_id "Bert-Slime-PCB:ICM-45686")
 		(at 152.4 140.97 0)
 		(unit 1)
@@
 		(dnp no)
 		(property "Reference" "U1"
-			(at 153.035 121.92 0)
-			(effects
-				(font
-					(size 1.27 1.27)
-				)
+			(at 111.76 99.568 0)
+			(effects
+				(font
+					(size 1.27 1.27)
+				)
+				(justify left bottom)
 			)
 		)
 		(property "Value" "ICM-45686"
-			(at 153.035 124.46 0)
-			(effects
-				(font
-					(size 1.27 1.27)
-				)
-			)
-		)
-		(property "Footprint" "ICM_45686:IC_ICM-45686"
-			(at 153.035 127 0)
-			(effects
-				(font
-					(size 1.27 1.27)
-				)
+			(at 128.016 152.146 0)
+			(effects
+				(font
+					(size 1.27 1.27)
+				)
+				(justify left top)
+			)
+		)
+		(property "Footprint" "Bert-Slime-PCB:IC_ICM-45686"
+			(at 153.67 153.416 0)
+			(effects
+				(font
+					(size 1.27 1.27)
+				)
+				(justify bottom)
 			)
 		)
@@
 	)
 	(symbol
-		(lib_id "SM05B-SRSS-TB-con:SM05B-SRSS-TB(LF)(SN)")
+		(lib_id "Bert-Slime-PCB:SM05B-SRSS-TB(LF)(SN)")
 		(at 241.3 92.71 0)
 		(unit 1)
@@
 			)
 		)
-		(property "Footprint" "Personal:CONN-SMD_SM05B-SRSS-TB-LF-SN"
+		(property "Footprint" "Bert-Slime-PCB:CONN-SMD_SM05B-SRSS-TB-LF-SN"
 			(at 241.3 105.41 0)
 			(effects
@@
 	)
 	(symbol
-		(lib_id "Personal_Library:D1_Mini")
+		(lib_id "Bert-Slime-PCB:D1_Mini")
 		(at 161.29 87.63 0)
 		(unit 1)
 		(exclude_from_sim no)
-		(in_bom no)
+		(in_bom yes)
 		(on_board yes)
 		(dnp no)
@@
 			)
 		)
-		(property "Footprint" "Personal:D1-Mini"
+		(property "Footprint" "Bert-Slime-PCB:D1-Mini"
 			(at 161.29 87.63 0)
 			(effects
@@
 	)
 	(symbol
-		(lib_id "PMEG3010ESBYL:PMEG3010ESBYL")
+		(lib_id "Bert-Slime-PCB:PMEG3010ESBYL")
 		(at 87.63 81.28 180)
 		(unit 1)
@@
 			)
 		)
-		(property "Footprint" "PMEG3010ESBYL:SOD993_L1.0-W0.6-LS1.0-RD"
+		(property "Footprint" "Bert-Slime-PCB:SOD993_L1.0-W0.6-LS1.0-RD"
 			(at 87.63 73.66 0)
 			(effects
@@
 	)
 	(symbol
-		(lib_id "MK-12C02-G020:MK-12C02-G020")
+		(lib_id "Bert-Slime-PCB:MK-12C02-G020")
 		(at 101.6 105.41 0)
 		(unit 1)
@@
 			)
 		)
-		(property "Footprint" "Personal:SW-SMD_MK-12C02-G020"
+		(property "Footprint" "Bert-Slime-PCB:SW-SMD_MK-12C02-G020"
 			(at 101.6 118.11 0)
 			(effects
@@
 	)
 	(symbol
-		(lib_id "kicad-library:TP4056-USBC-Module")
+		(lib_id "Bert-Slime-PCB:TP4056-USBC-Module")
 		(at 63.5 91.44 0)
 		(unit 1)
 		(exclude_from_sim no)
-		(in_bom no)
+		(in_bom yes)
 		(on_board yes)
 		(dnp no)
@@
 			)
 		)
-		(property "Footprint" "Personal:TP4056-USBC-MODULE"
+		(property "Footprint" "Bert-Slime-PCB:TP4056-USBC-MODULE"
 			(at 63.5 93.98 0)
 			(effects
@@
 	)
 	(symbol
-		(lib_id "PMEG3010ESBYL:PMEG3010ESBYL")
+		(lib_id "Bert-Slime-PCB:PMEG3010ESBYL")
 		(at 87.63 69.85 180)
 		(unit 1)
@@
 			)
 		)
-		(property "Footprint" "PMEG3010ESBYL:SOD993_L1.0-W0.6-LS1.0-RD"
+		(property "Footprint" "Bert-Slime-PCB:SOD993_L1.0-W0.6-LS1.0-RD"
 			(at 87.63 62.23 0)
 			(effects
@@
 	)
 	(symbol
-		(lib_id "Personal_Library:1532H-24.000JWVDTL")
+		(lib_id "Bert-Slime-PCB:1532H-24.000JWVDTL")
 		(at 77.47 139.7 0)
 		(unit 1)
@@
 		(dnp no)
 		(property "Reference" "Y1"
-			(at 77.47 122.428 0)
-			(effects
-				(font
-					(size 1.27 1.27)
-				)
+			(at 72.39 133.35 0)
+			(effects
+				(font
+					(size 1.27 1.27)
+				)
+				(justify left)
 			)
 		)
 		(property "Value" "1532H-24.000JWVDTL"
-			(at 77.47 124.968 0)
-			(effects
-				(font
-					(size 1.27 1.27)
-				)
-			)
-		)
-		(property "Footprint" "Personal:Crystal_SMD_3225-4Pin_3.2x2.5mm"
+			(at 78.74 146.05 0)
+			(effects
+				(font
+					(size 1.27 1.27)
+				)
+				(justify left)
+			)
+		)
+		(property "Footprint" "Crystal:Crystal_SMD_3225-4Pin_3.2x2.5mm"
 			(at 95.25 148.59 0)
 			(effects
